File: The Dichotomy Split/The Dichotomy Split.kicad_sch (KiCad schematic)
At the start: 0 parts

Commit message: Schematic AND pcb finished!
Parts:
- added H11, H12, H13: MountingHole, Panelization.pretty-master:mouse-bite-5mm-slot, symbol Mechanical:MountingHole
Other:
- added sheet left (side.kicad_sch)
- added sheet right (side.kicad_sch)
