File: The Dichotomy Split/The Dichotomy Split.kicad_pcb (KiCad board)
At the start: 2 copper layers, 265.9 x 99.6 mm, 149 parts, among them SW1 SW_Push, SW10 SW_Push, SW11 SW_Push, SW12 SW_Push, SW13 SW_Push, SW14 SW_Push, SW15 SW_Push, SW16 SW_Push, SW17 SW_Push, SW18 SW_Push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

Commit message: pictures CAD BOM GERBERS ZMK FIRMWARE
Parts:
- added G***: LOGO, LOGO, F.Cu at (210.7, 68.4)
- added G***: LOGO, LOGO, F.Cu at (99.3, 69.0)
Other:
- board text added: "By Cocotrilo - STASIS HackClub"
- board text added: "The Dichotomy Split"
